Commit message: minor

File: arm_controls/tests/mycobot_320pi.urdf (robot description, URDF)
Before this commit: robot firefighter, 7 links, 6 joints
Links:
- removed link base
- added link base_link; collision mesh filename=package://mycobot_description/urdf/mycobot_320_pi_2022/base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; visual mesh filename=package://mycobot_description/urdf/mycobot_320_pi_2022/base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
- added link gripper; visual box size=0.05 0.02 0.02
Joints:
- added joint wrist_to_gripper: type fixed, parent link6, child gripper, origin xyz=0.05 0 0 rpy=0 0 0
- joint joint2_to_joint1: parent base -> base_link

Commit message: minor

File: arm_controls/tests/mycobot_320pi.urdf (robot description, URDF)
Before this commit: robot firefighter, 8 links, 7 joints
Links:
- link gripper: geometry visual box size=0.158 0.105 0.055
