Commit message: minor

File: arm_controls/mycobot_320pi.urdf (robot description, URDF)
Before this commit: robot firefighter, 8 links, 7 joints
Joints:
- joint wrist_to_gripper: origin xyz=0.05 0 0 rpy=0 0 0 -> xyz=0.10 0 0 rpy=0 0 0

Commit message: urdf

File: arm_controls/mycobot_320pi.urdf (robot description, URDF)
Before this commit: robot firefighter, 8 links, 7 joints
Joints:
- joint wrist_to_gripper: origin xyz=0.10 0 0 rpy=0 0 0 -> xyz=0.05 0 0 rpy=0 0 0

Commit message: minor

File: arm_controls/mycobot_320pi.urdf (robot description, URDF)
Before this commit: robot firefighter, 8 links, 7 joints
Joints:
- joint wrist_to_gripper: origin xyz=0.05 0 0 rpy=0 0 0 -> xyz=0.11 0 0 rpy=0 0 0

Commit message: urdf

File: arm_controls/mycobot_320pi.urdf (robot description, URDF)
Before this commit: robot firefighter, 8 links, 7 joints
Joints:
- joint wrist_to_gripper: origin xyz=0.11 0 0 rpy=0 0 0 -> xyz=0 0 0.11 rpy=0 0 0

Commit message: minor

File: arm_controls/mycobot_320pi.urdf (robot description, URDF)
Before this commit: robot firefighter, 8 links, 7 joints
Joints:
- joint wrist_to_gripper: origin xyz=0 0 0.11 rpy=0 0 0 -> xyz=0 0 0.1 rpy=0 0 0

Commit message: urdf

File: arm_controls/mycobot_320pi.urdf (robot description, URDF)
Before this commit: robot firefighter, 8 links, 7 joints
Joints:
- joint wrist_to_gripper: origin xyz=0 0 0.1 rpy=0 0 0 -> xyz=0 0 0.12 rpy=0 0 0

Commit message: urdf

File: arm_controls/mycobot_320pi.urdf (robot description, URDF)
Before this commit: robot firefighter, 8 links, 7 joints
Joints:
- joint wrist_to_gripper: origin xyz=0 0 0.12 rpy=0 0 0 -> xyz=0 0 0.13 rpy=0 0 0

Commit message: minor

File: arm_controls/mycobot_320pi.urdf (robot description, URDF)
Before this commit: robot firefighter, 8 links, 7 joints
Links:
- link gripper: geometry visual box size=0.11 0.7 0.057

Commit message: removed offsets

File: arm_controls/mycobot_320pi.urdf (robot description, URDF)
Before this commit: robot firefighter, 8 links, 7 joints
Links:
- link gripper: geometry visual box xyz=0.045 0.05 0.13

Commit message: .urdf file

File: arm_controls/mycobot_320pi.urdf (robot description, URDF)
Before this commit: robot firefighter, 8 links, 7 joints
Links:
- link gripper: geometry visual box xyz=0.11 0.7 0.057
Joints:
- joint wrist_to_gripper: origin xyz=0 0 0.13 rpy=0 0 0 -> xyz=0.045 0.05 0.13 rpy=0 0 0

Commit message: urdf file

File: arm_controls/mycobot_320pi.urdf (robot description, URDF)
Before this commit: robot firefighter, 8 links, 7 joints
Links:
- link gripper: geometry visual box size=0.11 0.7 0.057
Joints:
- joint wrist_to_gripper: origin xyz=0.045 0.05 0.13 rpy=0 0 0 -> xyz=0 0 0.13 rpy=0 0 0

Commit message: minor

File: arm_controls/mycobot_320pi.urdf (robot description, URDF)
Before this commit: robot firefighter, 8 links, 7 joints
Links:
- link gripper: geometry visual box size=0.11 0.07 0.057

Commit message: active_links_mask

File: arm_controls/mycobot_320pi.urdf (robot description, URDF)
Before this commit: robot firefighter, 8 links, 7 joints
Joints:
- joint joint5_to_joint4: origin xyz=0.1205 0 0.082  rpy= 0 0 1.57080 -> xyz=0.1205 0 0 rpy= 0 0 1.57080
