Commit message: new urdf file

File: arm_controls/mycobot_320pi.urdf (robot description, URDF)
Before this commit: robot firefighter, 8 links, 7 joints
Links:
- link gripper: geometry visual box size=0 0 0
Joints:
- joint joint5_to_joint4: origin xyz=0.1205 0 0 rpy= 0 0 1.57080 -> xyz=0.1205 0 0.082 rpy= 0 0 1.57080
- joint wrist_to_gripper: origin xyz=0 0 0.13 rpy=0 0 0 -> xyz=0 0 0.07 rpy=0 0 0
